Commit message: Changed the geometry to align with the real robot

File: description/imu.xacro (robot description, xacro)
@@ -1,4 +1,7 @@
 <?xml version="1.0"?>
 <robot xmlns:xacro="http://www.ros.org/wiki/xacro"  name="imu_robot">
+  <material name="whites">
+      <color rgba="1 1 1 1" />
+  </material>
   <!-- IMU Sensor -->
   <link name="imu_link">
@@ -9,14 +12,12 @@
     </inertial>
     <visual>
-      <origin xyz="0 0 0"/>
+      <origin xyz="0 0 0.045"/>
       <geometry>
         <box size="0.02 0.02 0.02"/>
       </geometry>
-      <material>
-        <color rgba="0.0 1.0 0.0 1.0"/>
-      </material>
+      <material name="whites"/>
     </visual>
     <collision>
-      <origin xyz="0 0 0"/>
+      <origin xyz="0 0 0.045"/>
       <geometry>
         <box size="0.02 0.02 0.02"/>
@@ -27,5 +28,5 @@
     <parent link="base_link"/>
     <child link="imu_link"/>
-    <origin xyz="0 0 0.1" rpy="0 0 0"/>
+    <origin xyz="0 0 0.045" rpy="0 0 0"/>
   </joint>
   <gazebo reference="imu_link">

File: description/lidar.xacro (robot description, xacro)
@@ -4,10 +4,10 @@
     <parent link="chassis"/>
     <child link="laser_frame" />
-    <origin xyz="0.1 0 0.175" rpy="0 0 0"/>
+    <origin xyz="0 0 0.110" rpy="0 0 0"/>
   </joint>
   <link name="laser_frame">
     <visual>
         <geometry>
-            <cylinder radius="0.05" length="0.04"/>
+            <cylinder radius="0.035" length="0.05"/>
         </geometry>
         <material name="red"/>
@@ -15,8 +15,8 @@
     <collision>
         <geometry>
-            <cylinder radius="0.05" length="0.04"/>
+            <cylinder radius="0.035" length="0.05"/>
         </geometry>
     </collision>
-    <xacro:inertial_cylinder mass="0.1" length="0.04" radius="0.05">
+    <xacro:inertial_cylinder mass="0.1" length="0.05" radius="0.035">
         <origin xyz="0 0 0" rpy="0 0 0"/>
     </xacro:inertial_cylinder>

File: description/robot_core.xacro (robot description, xacro)
@@ -31,24 +31,43 @@
         <parent link="base_link"/>
         <child link="chassis"/>
-        <origin xyz="-0.1 0 0"/>
+        <origin xyz="0 0 0"/>
     </joint>
-    <link name="chassis">
-        <visual>
-            <origin xyz="0.15 0 0.075"/>
-            <geometry>
-                <box size="0.3 0.3 0.15"/>
-            </geometry>
-            <material name="white"/>
-        </visual>
-        <collision>
-            <origin xyz="0.15 0 0.075"/>
-            <geometry>
-                <box size="0.3 0.3 0.15"/>
-            </geometry>
-        </collision>
-        <xacro:inertial_box mass="0.5" x="0.3" y="0.3" z="0.15">
-            <origin xyz="0.15 0 0.075" rpy="0 0 0"/>
-        </xacro:inertial_box>
-    </link>
+  <link name="chassis">
+      <visual>
+          <origin xyz="0 0 0.065"/> <!-- half the height (90mm) is 45mm, plus 20mm above ground -->
+          <geometry>
+              <cylinder radius="0.1" length="0.09"/>
+          </geometry>
+          <material name="white"/>
+      </visual>
+      <collision>
+          <origin xyz="0 0 0.065"/>
+          <geometry>
+              <cylinder radius="0.1" length="0.09"/>
+          </geometry>
+      </collision>
+      <xacro:inertial_cylinder mass="0.5" radius="0.1" length="0.09">
+          <origin xyz="0 0 0.065" rpy="0 0 0"/>
+      </xacro:inertial_cylinder>
+  </link>
+    <!-- <link name="chassis"> -->
+    <!--     <visual> -->
+    <!--         <origin xyz="0.15 0 0.075"/> -->
+    <!--         <geometry> -->
+    <!--             <box size="0.3 0.3 0.15"/> -->
+    <!--         </geometry> -->
+    <!--         <material name="white"/> -->
+    <!--     </visual> -->
+    <!--     <collision> -->
+    <!--         <origin xyz="0.15 0 0.075"/> -->
+    <!--         <geometry> -->
+    <!--             <box size="0.3 0.3 0.15"/> -->
+    <!--         </geometry> -->
+    <!--     </collision> -->
+    <!--     <xacro:inertial_box mass="0.5" x="0.3" y="0.3" z="0.15"> -->
+    <!--         <origin xyz="0.15 0 0.075" rpy="0 0 0"/> -->
+    <!--     </xacro:inertial_box> -->
+    <!-- </link> -->
+    <!---->
     <gazebo reference="chassis">
       <material>Gazebo/White</material>
@@ -58,5 +77,5 @@
         <parent link="base_link"/>
         <child link="left_wheel"/>
-        <origin xyz="0 0.175 0" rpy="-${pi/2} 0 0" />
+        <origin xyz="0 0.1015 0" rpy="-${pi/2} 0 0" />
         <axis xyz="0 0 1"/>
     </joint>
@@ -64,5 +83,5 @@
         <visual>
             <geometry>
-                <cylinder radius="0.05" length="0.04"/>
+                <cylinder radius="0.035" length="0.035"/>
             </geometry>
             <material name="blue"/>
@@ -70,8 +89,8 @@
         <collision>
             <geometry>
-                <sphere radius="0.05"/>
+                <sphere radius="0.035"/>
             </geometry>
         </collision>
-        <xacro:inertial_cylinder mass="0.1" length="0.04" radius="0.05">
+        <xacro:inertial_cylinder mass="0.1" length="0.035" radius="0.035">
             <origin xyz="0 0 0" rpy="0 0 0"/>
         </xacro:inertial_cylinder>
@@ -84,5 +103,5 @@
         <parent link="base_link"/>
         <child link="right_wheel"/>
-        <origin xyz="0 -0.175 0" rpy="${pi/2} 0 0" />
+        <origin xyz="0 -0.1015 0" rpy="${pi/2} 0 0" />
         <axis xyz="0 0 -1"/>
     </joint>
@@ -90,5 +109,5 @@
         <visual>
             <geometry>
-                <cylinder radius="0.05" length="0.04"/>
+                <cylinder radius="0.035" length="0.035"/>
             </geometry>
             <material name="blue"/>
@@ -96,8 +115,8 @@
         <collision>
             <geometry>
-                <sphere radius="0.05"/>
+                <sphere radius="0.035"/>
             </geometry>
         </collision>
-        <xacro:inertial_cylinder mass="0.1" length="0.04" radius="0.05">
+        <xacro:inertial_cylinder mass="0.1" length="0.035" radius="0.035">
             <origin xyz="0 0 0" rpy="0 0 0"/>
         </xacro:inertial_cylinder>
@@ -110,10 +129,10 @@
         <parent link="chassis"/>
         <child link="caster_wheel"/>
-        <origin xyz="0.24 0 0"/>
+        <origin xyz="0.09 0 0"/>
     </joint>
     <link name="caster_wheel">
         <visual>
             <geometry>
-                <sphere radius="0.05"/>
+                <sphere radius="0.028"/>
             </geometry>
             <material name="black"/>
@@ -121,8 +140,29 @@
         <collision>
             <geometry>
-                <sphere radius="0.05"/>
+                <sphere radius="0.028"/>
             </geometry>
         </collision>
-        <xacro:inertial_sphere mass="0.1" radius="0.05">
+        <xacro:inertial_sphere mass="0.1" radius="0.028">
+            <origin xyz="0 0 0" rpy="0 0 0"/>
+        </xacro:inertial_sphere>
+    </link>
+    <joint name="caster_wheel_joint2" type="fixed">
+        <parent link="chassis"/>
+        <child link="caster_wheel2"/>
+        <origin xyz="-0.09 0 0"/>
+    </joint>
+    <link name="caster_wheel2">
+        <visual>
+            <geometry>
+                <sphere radius="0.028"/>
+            </geometry>
+            <material name="black"/>
+        </visual>
+        <collision>
+            <geometry>
+                <sphere radius="0.028"/>
+            </geometry>
+        </collision>
+        <xacro:inertial_sphere mass="0.1" radius="0.028">
             <origin xyz="0 0 0" rpy="0 0 0"/>
         </xacro:inertial_sphere>
@@ -133,3 +173,8 @@
       <mu2 value="0.001"/>
     </gazebo>
+    <gazebo reference="caster_wheel2">
+      <material>Gazebo/Black</material>
+      <mu1 value="0.001"/>
+      <mu2 value="0.001"/>
+    </gazebo>
 </robot>
