Commit message: wheels correct size and postion, lidar output remapping, changed spawn of robot

File: description/lidar.xacro (robot description, xacro)
@@ -26,5 +26,5 @@
     <sensor name="laser" type="ray">
       <pose> 0 0 0 0 0 0 </pose>
-      <visualize> false </visualize>
+      <visualize> true </visualize>
       <update_rate>10</update_rate>
       <ray>
@@ -45,5 +45,6 @@
       <plugin name="laser_controller" filename="libgazebo_ros_ray_sensor.so">
         <ros>
-          <argument>--ros-args --remap ~/out:=scan</argument>
+          <namespace>/</namespace>
+          <remapping>laser_controller/out:=scan</remapping>
         </ros>
         <output_type>sensor_msgs/LaserScan</output_type>

File: description/robot_core.xacro (robot description, xacro)
@@ -77,5 +77,5 @@
         <parent link="base_link"/>
         <child link="left_wheel"/>
-        <origin xyz="0 0.1015 0" rpy="-${pi/2} 0 0" />
+        <origin xyz="0 0.1175 0" rpy="-${pi/2} 0 0" />
         <axis xyz="0 0 1"/>
     </joint>
@@ -103,5 +103,5 @@
         <parent link="base_link"/>
         <child link="right_wheel"/>
-        <origin xyz="0 -0.1015 0" rpy="${pi/2} 0 0" />
+        <origin xyz="0 -0.1175 0" rpy="${pi/2} 0 0" />
         <axis xyz="0 0 -1"/>
     </joint>
@@ -134,5 +134,5 @@
         <visual>
             <geometry>
-                <sphere radius="0.028"/>
+                <sphere radius="0.035"/>
             </geometry>
             <material name="black"/>
@@ -140,8 +140,8 @@
         <collision>
             <geometry>
-                <sphere radius="0.028"/>
+                <sphere radius="0.035"/>
             </geometry>
         </collision>
-        <xacro:inertial_sphere mass="0.1" radius="0.028">
+        <xacro:inertial_sphere mass="0.1" radius="0.035">
             <origin xyz="0 0 0" rpy="0 0 0"/>
         </xacro:inertial_sphere>
@@ -155,5 +155,5 @@
         <visual>
             <geometry>
-                <sphere radius="0.028"/>
+                <sphere radius="0.035"/>
             </geometry>
             <material name="black"/>
@@ -161,8 +161,8 @@
         <collision>
             <geometry>
-                <sphere radius="0.028"/>
+                <sphere radius="0.035"/>
             </geometry>
         </collision>
-        <xacro:inertial_sphere mass="0.1" radius="0.028">
+        <xacro:inertial_sphere mass="0.1" radius="0.035">
             <origin xyz="0 0 0" rpy="0 0 0"/>
         </xacro:inertial_sphere>
