Commit message: update

File: description/ros2_control.xacro (robot description, xacro)
@@ -1,4 +1,44 @@
 <?xml version="1.0"?>
 <robot xmlns:xacro="http://www.ros.org/wiki/xacro" >
+  <ros2_control name="RealRobot" type="system">
+    <hardware>
+	<plugin>diffbot_arduino/DiffDriveArduino</plugin>
+	<param name="left_wheel_name">left_wheel_joint</param>
+        <param name="right_wheel_name">right_wheel_joint</param>
+        <param name="loop_rate">30</param>
+        <param name="device">/dev/serial/by-id/usb-Silicon_Labs_CP2102_USB_to_UART_Bridge_Controller_0001-if00-port0</param>
+        <param name="baud_rate">57600</param>
+        <param name="timeout">1000</param>
+        <param name="enc_counts_per_rev">2597</param>
+    </hardware>
+    <joint name="left_wheel_joint">
+      <command_interface name="velocity">
+        <param name="min">-10</param>
+        <param name="max">10</param>
+      </command_interface>
+      <state_interface name="velocity"/>
+      <state_interface name="position"/>
+    </joint>
+    <joint name="right_wheel_joint">
+      <command_interface name="velocity">
+        <param name="min">-10</param>
+        <param name="max">10</param>
+      </command_interface>
+      <state_interface name="velocity"/>
+      <state_interface name="position"/>
+    </joint>
+    <!--    <sensor name="imu_sensor" type="imu_sensor">
+      <state_interface name="orientation.x"/>
+      <state_interface name="orientation.y"/>
+      <state_interface name="orientation.z"/>
+      <state_interface name="orientation.w"/>
+      <state_interface name="angular_velocity.x"/>
+      <state_interface name="angular_velocity.y"/>
+      <state_interface name="angular_velocity.z"/>
+      <state_interface name="linear_acceleration.x"/>
+      <state_interface name="linear_acceleration.y"/>
+      <state_interface name="linear_acceleration.z"/>
+    </sensor>
+  </ros2_control>
   <ros2_control name="DiffBotSystem" type="system">
     <hardware>
@@ -21,5 +61,4 @@
       <state_interface name="position"/>
     </joint>
-        <!-- IMU Sensor Interface -->
     <sensor name="imu_sensor" type="imu_sensor">
       <state_interface name="orientation.x"/>
@@ -39,4 +78,4 @@
       <parameters>$(find diffbot)/config/ros2_controller.yaml</parameters>
     </plugin>
-  </gazebo>
+  </gazebo> -->
 </robot>
