Commit message: need to use gz_ros2_control and not gazebo plugin

File: diffbot/description/lidar.xacro (robot description, xacro)
@@ -1,6 +1,7 @@
 <?xml version="1.0"?>
 <robot xmlns:xacro="http://www.ros.org/wiki/xacro" >
+  <xacro:include filename="inertial_macros.xacro"/>
   <joint name="laser_joint" type="fixed">
-    <parent link="chassis"/>
+    <parent link="base_link"/>
     <child link="laser_frame" />
     <origin xyz="0 0 0.110" rpy="0 0 0"/>
@@ -11,5 +12,4 @@
             <cylinder radius="0.035" length="0.05"/>
         </geometry>
-        <material name="red"/>
     </visual>
     <collision>
