Commit message: Removing gazebo references and adding them to the world file

File: diffbot/description/urdf/diffbot.urdf (robot description, URDF)
Before this commit: robot robot, 9 links, 7 joints
Links:
- removed link LidarLink
- added link base_scan, mass 0.025133; collision mesh filename=package://diffbot/meshes/collision/LidarLink.STL; visual mesh filename=package://diffbot/meshes/visual/LidarLink.STL
Joints:
- removed joint lidar_joint
- added joint scan_joint: type fixed, parent base_link, child base_scan, origin xyz=0 0 0.056 rpy=0 0 0
- joint left_wheel_joint: limit lower=-3.14 upper=3.14 effort=10 velocity=10 -> (none); type revolute -> continuous
- joint right_wheel_joint: limit lower=-3.14 upper=3.14 effort=10 velocity=10 -> (none); type revolute -> continuous

Commit message: save

File: diffbot/description/urdf/diffbot.urdf (robot description, URDF)
Before this commit: robot robot, 9 links, 7 joints
Links:
- removed link base_footprint
- removed link laser_frame
Joints:
- removed joint laser_joint
